File: hw/pesho.sch (KiCad schematic (older format))
At the start: 0 parts

Commit message: more hw files
Parts:
- added B?: BKS-300, symbol BKS-300
- added C? (x5): 100n, symbol C
- added C?: 1u, symbol C
- added C? (x2): C, symbol C
- added M?: L298P-BREAKOUT, symbol L298P-BREAKOUT
- added Q?: BUCK5V, symbol BUCK5V
- added R? (x3): 330k, symbol R
- added R? (x3): 510, symbol R
- added R? (x2): 10k, symbol R
- added RPi?: RPI_B+, symbol RPI_B+
- added SW? (x2): SPST, symbol SPST
- added U? (x3): OPTO-TRANSISTOR, symbol OPTO-TRANSISTOR
Connections:
- net labels added: +12V, +3.3V, +5V, BD, BD_IN, BLK, BLK_IN, BUK, BUK_IN, EN_MOTOR_OUT, GND, LOCK_OUT, UNLOCK_OUT
- wire segments 0 -> 92
