File: hardware/pesho.sch (KiCad schematic (older format))
At the start: 32 parts

Commit message: moved stuff around
Parts:
- gave numbers to parts that had none: 32
Connections:
- wire segments 117 -> 120
